File: MCU/MCU.kicad_sch (KiCad schematic)
At the start: 40 parts, among them J1 Screw_Terminal_2x5.08, U1 INA597IDR, U2 INA597IDR, U3 NUCLEO144-F767ZI, U4 INA597IDR, U5 INA597IDR, U6 INA597IDR

Commit message: current sensors
Parts:
- removed J1: Screw_Terminal_2x5.08, rsx_headers_screw:Molex_0398800302, symbol rsx_header_screw:Screw_Terminal_2x5.08
- added C11, C12, C13: 0u1, rsx_capacitors:C_0603_1608Metric, symbol rsx_Capacitors:0u1
- added C14: 1u, rsx_capacitors:C_0805_2012Metric, symbol rsx_Capacitors:1u
- added R20, R21, R23: 200R_2W, rsx_resistors:R_2512_6332Metric, symbol rsx_Resistors:200R_2W
- added R22: 330R, rsx_resistors:R_0603_1608Metric, symbol rsx_Resistors:330R
- added R24: 100K 0.1%, rsx_resistors:R_0603_1608Metric, symbol rsx_Resistors:100K 0.1%
- added U7: 200A_AC_HALL_ALLEGRO, rsx_packages_SO:SOIC-8_3.9x4.9mm_P1.27mm_DL, symbol rsx_sensors:200A_AC_HALL_ALLEGRO_1
- added U8: 30A_AC_HALL_ALLEGRO, rsx_packages_SO:SOIC-8_3.9x4.9mm_P1.27mm_DL, symbol rsx_sensors:30A_AC_HALL_ALLEGRO_1
Connections:
- net 5V: now also C11.2, U7.1 (VCC)
- net GND: now also C11.1, C12.2, C13.2, C14.2, U7.2 (GND), U7.4 (NC), U7.7 (NC), U8.5 (GND)
- net at D2.2 (A): now also R21.2
- net 30A_meas: now reaches U3.110 (PF4)
- net 30A_meas: now also C14.1, U8.7 (VIOUT)
- net 150A_meas: now reaches U3.114 (PF10)
- net 150A_meas: now also C12.1, U7.3 (VIOUT)
- net Green: now reaches U3.133 (PG14)
- net Green: now also R21.1
- net 3.3V: now reaches U3.16 (+3V3)
- net 3.3V: now also C13.1, R24.1, U8.8 (VCC)
- net BLUE: now reaches U3.63 (PG9)
- net BLUE: now also R20.1
- net RED: now reaches U3.64 (PG15)
- net RED: now also R22.1
- net YELLOW: now reaches U3.68 (PG13/ETH_TXD0)
- net YELLOW: now also R23.1
- net at D4.2 (A): now also R23.2
- net at D3.2 (A): now also R22.2
- net at D1.2 (A): now also R20.2
- new net: R24.2, U8.6 (FAULT)
- new net 150A_Current_IN: U7.5 (IP+)
- new net 150A_Current_OUT: U7.6 (IP-)
- new net 30A_Current_IN: U8.1 (IP+), U8.2 (IP+)
- new net 30A_Current_OUT: U8.3 (IP-), U8.4 (IP-)
Other:
- moved on the sheet: D1, D2, D3, D4
