File: MCU/MCU.kicad_sch (KiCad schematic)
At the start: 66 parts, among them J1 Screw_Terminal_2x2.54, J2 Screw_Terminal_2x2.54, J3 Screw_Terminal_2x2.54, J4 Screw_Terminal_2x2.54, Q1 2N7002K, Q2 2N7002K, Q3 2N7002K, Q4 2N7002K, Q5 2N7002K, U1 INA597IDR, U2 INA597IDR, U3 NUCLEO144-F767ZI, U4 INA597IDR, U5 INA597IDR, U6 INA597IDR, U7 200A_AC_HALL_ALLEGRO, U8 30A_AC_HALL_ALLEGRO

Commit message: hi
Parts:
- removed D1: LED_B, rsx_leds:LED_0805_2012Metric, symbol rsx_LEDs:LED_B
- removed D3: LED_R, rsx_leds:LED_0805_2012Metric, symbol rsx_LEDs:LED_R
- removed D4: LED_Y, rsx_leds:LED_0805_2012Metric, symbol rsx_LEDs:LED_Y
- removed Q1, Q3, Q4, Q5: 2N7002K, rsx_packages_TO_SOT:SOT-23, symbol rsx_Transistors:2N7002K
- removed R16, R17, R18, R19: 0R100 1/2W, rsx_resistors:R_1206_3216Metric, symbol rsx_Resistors:0R100 1/2W
- removed R20, R21, R23: 200R_2W, rsx_resistors:R_2512_6332Metric, symbol rsx_Resistors:200R_2W
- added D1, D10, D3, D4: LED_G, rsx_leds:LED_0805_2012Metric, symbol rsx_LEDs:LED_G
- added D6, D7, D8, D9: LED_B, rsx_leds:LED_0805_2012Metric, symbol rsx_LEDs:LED_B
- added J5: Screw_Terminal_2x2.54, rsx_headers_screw:Wurth_691210910002, symbol rsx_header_screw:Screw_Terminal_2x2.54
- added K1: G5LE-1_12V, rsx_relays:Relay_SPDT_Omron-G5LE-1, symbol rsx_Relays:G5LE-1_12V
- added Q1, Q3, Q4, Q6: RXH090N03, rsx_packages_SO:SOIC-8_3.9x4.9mm_P1.27mm_DL, symbol rsx_Transistors:RXH090N03
- added Q7: 2N7002K, rsx_packages_TO_SOT:SOT-23, symbol rsx_Transistors:2N7002K
- added R16, R17, R18, R19, R20, R21, R23, R30: 330R, rsx_resistors:R_0603_1608Metric, symbol rsx_Resistors:330R
- added R31, R32, R33, R34, R35, R36, R37, R38: 100R, rsx_resistors:R_0603_1608Metric, symbol rsx_Resistors:100R
- added SW1: Button, rsx_HID:FSMSMTR, symbol rsx_HID:Button
- added U10, U11, U12, U9: -40C-125C, rsx_packages_TO_SOT:SOT-23, symbol rsx_sensors:MCP9700A-E/TO
Connections:
- net 12V: no longer J1.2 (Pin_2), J2.2 (Pin_2), J3.2 (Pin_2), J4.2 (Pin_2)
- net 3.3V: now also U10.1 (VCC), U11.1 (VCC), U12.1 (VCC), U9.1 (VCC)
- net ENA_Boost(19V): now also R16.1, R32.2
- net ENA_Boost(24V): now also R18.1, R34.2
- net ENA_Boost(56V): now also R17.1, R33.2
- net ENA_Buck(12V): now also R30.1, R31.2
- net GND: now also D1.1 (K), D10.1 (K), D3.1 (K), D6.1 (K), D7.1 (K), D8.1 (K), D9.1 (K), Q1.1 (S), Q1.2 (S), Q1.3 (S), Q3.1 (S), Q3.2 (S), Q3.3 (S), Q4.1 (S), Q4.2 (S), Q4.3 (S), Q6.1 (S), Q6.2 (S), Q6.3 (S), Q7.2 (S), SW1.2, U10.3 (GND), U11.3 (GND), U12.3 (GND), U9.3 (GND)
- net RED: no longer R22.1
- net fan1_EN: now also R21.1, R37.2; no longer U3.75 (PB8)
- net fan2_EN: now also R22.1, R38.2; no longer U3.77 (PB9)
- net fan3_EN: now also R19.1, R35.2; no longer U3.118 (PD14)
- net fan4_EN: now also R20.1, R36.2; no longer U3.120 (PD15)
- net at U3.103 (SWO/PB3): now also R34.1
- net at R25.2: now also Q6.4 (G)
- net at J1.1 (Pin_1): now also Q6.5 (D), Q6.6 (D), Q6.7 (D), Q6.8 (D)
- net at R28.2: now also Q4.4 (G)
- net at J3.1 (Pin_1): now also Q4.5 (D), Q4.6 (D), Q4.7 (D), Q4.8 (D)
- net at R29.2: now also Q1.4 (G)
- net at J4.1 (Pin_1): now also Q1.5 (D), Q1.6 (D), Q1.7 (D), Q1.8 (D)
- net at R22.2: now also D3.2 (A)
- net at D2.2 (A): now also R21.2
- net at U3.94 (PB2): now also R33.1
- net TempMes3: now reaches U3.11 (PF7)
- net TempMes3: now also U11.2 (VOUT)
- net at U3.34 (PB0): now also R31.1
- net TempMes2: now reaches U3.54 (PF8)
- net TempMes2: now also U10.2 (VOUT)
- net TempMes4: now reaches U3.56 (PF9)
- net TempMes4: now also U12.2 (VOUT)
- net !E-STOP: now reaches U3.85 (PA6)
- net !E-STOP: now also Q7.1 (G)
- net TempMes1: now reaches U3.87 (ETH_CRS_DV/PA7)
- net TempMes1: now also U9.2 (VOUT)
- net at U3.96 (PB1): now also R32.1
- net at R27.2: now also Q3.4 (G)
- net at J2.1 (Pin_1): now also Q3.5 (D), Q3.6 (D), Q3.7 (D), Q3.8 (D)
- new net: D10.2 (A), R20.2
- new net: D4.1 (K), SW1.1
- new net: D4.2 (A), R23.2
- new net: D7.2 (A), R16.2
- new net: J5.1 (Pin_1), K1.3
- new net: R37.1, U3.75 (PB8)
- new net: D9.2 (A), R18.2
- new net: K1.5, Q7.3 (D), R23.1
- new net: D1.2 (A), R19.2
- new net: R38.1, U3.77 (PB9)
- new net: D6.2 (A), R30.2
- new net: D8.2 (A), R17.2
- new net: R35.1, U3.118 (PD14)
- new net: R36.1, U3.120 (PD15)
- new net +12V: J1.2 (Pin_2), J2.2 (Pin_2), J3.2 (Pin_2), J4.2 (Pin_2), K1.2
- new net V_BAT+: J5.2 (Pin_2), K1.1
- no-connect marks 0 -> 1
